File: reveil.kicad_pcb (KiCad board)
At the start: 2 copper layers, 170 x 90 mm, 38 parts, among them J1 Barrel_Jack_Switch, J2 AudioJack3_SwitchTR, Q1 2N3904, Q2 IRLB8721PBF, U1 MAX7219, U2 MAX7219

Commit message: cosmetic
Parts:
- added REF**: OSHW-Logo2_7.3x6mm_SilkScreen, Symbol:OSHW-Logo2_7.3x6mm_SilkScreen, F.Cu at (219.5, 99.0)
- added REF**: KiCad-Logo2_5mm_SilkScreen, Symbol:KiCad-Logo2_5mm_SilkScreen, F.Cu at (222.5, 105.0)
